Commit message: Cambio de robot a ur3e

File: ur_ws/src/easy_ur_control/urdf/ur_wrapper.xacro (robot description, xacro)
@@ -36,5 +36,5 @@
         visual_parameters_file="$(arg visual_parameters_file)"
     >
-        <origin xyz="0.460 0.436 0.910" rpy="3.14159 0 0" />
+        <origin xyz="0.180 -0.274 0.116" rpy="0 0 3.14159" />
     </xacro:ur_robot>
     <xacro:ur_ros2_control
